File: high-side-switch.kicad_sch (KiCad schematic)
At the start: 5 parts, among them Q2 BC847, Q3 BC856

Commit message: Final workings
Parts:
- Q2: value BC847 -> BC846
Changed lines of the file:
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@@
 			)
 		)
-		(property "Value" "BC847"
+		(property "Value" "BC846"
 			(at 125.73 109.2199 0)
 			(effects
